Commit message: monoped with xpp

File: urdf_dev/3_link_arm/3_link_arm.xacro (robot description, xacro)
@@ -4,7 +4,7 @@
   <xacro:property name="arm_link_radius" value="0.02"/>
   <xacro:include filename="$(find urdf_dev)/macros.xacro"/>
-  <xacro:include filename="$(find urdf_dev)/3_link_arm.gazebo"/>
+  <xacro:include filename="$(find urdf_dev)/3_link_arm/3_link_arm.gazebo"/>
   <!-- give a name to prevent link/joint names overlapping -->
-  <xacro:macro name="3DOF_joint" params="name parent child *origin">
+  <xacro:macro name="ball_joint" params="name parent child *origin">
     <joint name="${name}_fixed_joint" type="fixed">
         <xacro:insert_block name="origin"/>
@@ -74,7 +74,7 @@
     </xacro:cylinder_inertial>
   </link>
-  <xacro:3DOF_joint name="arm_base" parent="base_link" child="arm_link1">
-    <origin xyz="0 0 ${chassis_length/2}" rpy="0 0 0"/>
-  </xacro:3DOF_joint>
+  <xacro:ball_joint name="arm_base" parent="base_link" child="arm_link1">
+    <origin xyz="0 0 0" rpy="0 0 0"/>
+  </xacro:ball_joint>
   <link name="arm_link2">
     <visual>

File: urdf_dev/box_2wheel_base/box_2wheel_base.xacro (robot description, xacro)
@@ -1,10 +1,11 @@
 <?xml version='1.0'?>
-<robot name="cylinder_2wheel_base" xmlns:xacro="http://www.ros.org/wiki/xacro">
-  <xacro:property name="chassis_length" value="0.06"/>
-  <xacro:property name="chassis_radius" value="0.2"/>
-  <xacro:property name="wheel_length" value="0.04"/>
-  <xacro:property name="wheel_radius" value="0.07"/>
+<robot name="box_2wheel_base" xmlns:xacro="http://www.ros.org/wiki/xacro">
+  <xacro:property name="chassis_x" value="0.4"/>
+  <xacro:property name="chassis_y" value="0.2"/>
+  <xacro:property name="chassis_z" value="0.1"/>
+  <xacro:property name="wheel_length" value="0.05"/>
+  <xacro:property name="wheel_radius" value="0.11"/>
   <xacro:include filename="$(find urdf_dev)/macros.xacro"/>
-  <xacro:include filename="$(find urdf_dev)/cylinder_2wheel_base/cylinder_2wheel_base.gazebo"/>
+  <xacro:include filename="$(find urdf_dev)/box_2wheel_base/box_2wheel_base.gazebo"/>
   <!-- prefix:left reflect:-1 -->
   <xacro:macro name="wheel" params="prefix reflect">
@@ -31,5 +32,5 @@
       <parent link="chassis"/>
       <child link="${prefix}_wheel"/>
-      <origin xyz="0 ${reflect*chassis_radius} ${wheel_radius}"/>
+      <origin xyz="${chassis_x/4} ${reflect*chassis_y} ${wheel_radius}"/>
       <axis xyz="0 1 0" rpy="0 0 0"/>
       <!--limit effort="10000" velocity="1000"/-->
@@ -37,11 +38,26 @@
     </joint>
   </xacro:macro>
-  <!-- reflect:-1(back) -->
-  <xacro:macro name="caster" params="reflect">
+  <link name="chassis">
     <visual>
       <geometry>
-        <sphere radius="${(wheel_radius-chassis_length/2)/2}"/>
+        <cylinder length="${chassis_z}" radius="${chassis_y}"/>
       </geometry>
-      <origin xyz="${reflect*chassis_radius/1.33} 0 ${(wheel_radius-chassis_length/2)/2}" rpy="0 0 0"/>
+      <origin xyz="0 0 ${wheel_radius}" rpy="0 0 0"/>
+      <material name="black"/>
+    </visual>
+    <collision>
+      <geometry>
+        <cylinder length="${chassis_z}" radius="${chassis_y}"/>
+      </geometry>
+      <origin xyz="0 0 ${wheel_radius}" rpy="0 0 0"/>
+    </collision>
+    <xacro:cylinder_inertial m="${3.14*chassis_y*chassis_y*chassis_z}" r="${chassis_y}" l="${chassis_z}">
+      <origin xyz="0 0 ${wheel_radius}" rpy="0 0 0"/>
+    </xacro:cylinder_inertial>
+    <visual>
+      <geometry>
+        <sphere radius="${wheel_radius-chassis_z}"/>
+      </geometry>
+      <origin xyz="${-chassis_x/4} 0 ${wheel_radius-chassis_z}" rpy="0 0 0"/>
     </visual>
     <collision>
@@ -49,5 +65,5 @@
         <sphere radius="${wheel_radius/2}"/>
       </geometry>
-      <origin xyz="${reflect*chassis_radius/1.33} 0 ${(wheel_radius-chassis_length/2)/2}" rpy="0 0 0"/>
+      <origin xyz="${-chassis_x/4} 0 ${wheel_radius-chassis_z}" rpy="0 0 0"/>
       <surface>
         <friction>
@@ -63,26 +79,6 @@
     <!-- 0.523599 ~= pi * 4/3 / 8 -->
     <xacro:sphere_inertial m="${0.523599*wheel_radius*wheel_radius*wheel_radius}" r="${wheel_radius/2}">
-      <origin xyz="${reflect*chassis_radius/1.33} 0 ${(wheel_radius-chassis_length/2)/2}" rpy="0 0 0"/>
+      <origin xyz="${-chassis_x/4} 0 ${wheel_radius-chassis_z}" rpy="0 0 0"/>
     </xacro:sphere_inertial>
-  </xacro:macro>
-  <link name="chassis">
-    <visual>
-      <geometry>
-        <cylinder length="${chassis_length}" radius="${chassis_radius}"/>
-      </geometry>
-      <origin xyz="0 0 ${wheel_radius}" rpy="0 0 0"/>
-      <material name="black"/>
-    </visual>
-    <collision>
-      <geometry>
-        <cylinder length="${chassis_length}" radius="${chassis_radius}"/>
-      </geometry>
-      <origin xyz="0 0 ${wheel_radius}" rpy="0 0 0"/>
-    </collision>
-    <xacro:cylinder_inertial m="${3.14*chassis_radius*chassis_radius*chassis_length}" r="${chassis_radius}" l="${chassis_length}">
-      <origin xyz="0 0 ${wheel_radius}" rpy="0 0 0"/>
-    </xacro:cylinder_inertial>
-    <xacro:caster reflect="-1"/>
-    <xacro:caster reflect="1"/>
   </link>
   <xacro:wheel prefix="left" reflect="-1"/>
